Commit message: world added and buffing tool stl added

File: fanuc_gazebo/urdf/rot_base.xacro (robot description, xacro)
@@ -1,9 +1,9 @@
 <?xml version="1.0"?>
-<robot name="base_bot"  xmlns:xacro="http://ros.org/wiki/xacro">
-    <link name="world"/>
-<joint name="world_joint" type="fixed">
+<robot name="fanuc"  xmlns:xacro="http://ros.org/wiki/xacro">
+    <!-- <link name="world"/> -->
+<joint name="world_joint_2" type="fixed">
     <parent link="world" />
     <child link = "base_blob" />
-    <origin xyz="1.5 0 0" rpy="0.0 0.0 0" />
+    <origin xyz="2.0 0 0" rpy="0.0 0.0 0" />
 </joint>
     <link name="base_blob">
@@ -31,6 +31,6 @@
 </link>
 <joint name="main_joint" type="revolute">
-      <parent link="base_link" />
-      <child link = "link_1" />
+      <parent link="base_blob" />
+      <child link = "rot_blob" />
       <origin xyz="0 0 0.62" rpy="0.0 0.0 0.0" />
       <axis xyz="0 0 1" />
@@ -60,3 +60,19 @@
       </collision>
 </link>
+<!-- <transmission name="main_joint_tran">
+    <type>transmission_interface/SimpleTransmission</type>
+    <joint name="main_joint">
+      <hardwareInterface>hardware_interface/EffortJointInterface</hardwareInterface>
+    </joint>
+    <actuator name="main_joint_motor">
+      <hardwareInterface>hardware_interface/EffortJointInterface</hardwareInterface>
+      <mechanicalReduction>1</mechanicalReduction>
+    </actuator>
+</transmission> -->
+<!--
+<gazebo>
+      <plugin name="gazebo_ros_control" filename="libgazebo_ros_control.so">
+         <robotSimType>gazebo_ros_control/DefaultRobotHWSim</robotSimType>
+      </plugin>
+   </gazebo> -->
 </robot>
