Commit message: Added: f/t sensor added

File: fanuc_gazebo/urdf/arm_new.xacro (robot description, xacro)
@@ -5,5 +5,5 @@
     <parent link="world" />
     <child link = "base_link" />
-    <origin xyz="0 0 0.3" rpy="0.0 0.0 0" />
+    <origin xyz="0 0 0" rpy="0.0 0.0 0" />
 </joint>
 <link name="base_link">
@@ -230,4 +230,15 @@
       <child link="tool0" />
     </joint>
+<!-- Force Torque sensor -->
+<gazebo reference="joint_6">
+      <provideFeedback>true</provideFeedback>
+  </gazebo>
+  <gazebo>
+      <plugin name="ft_sensor" filename="libgazebo_ros_ft_sensor.so">
+          <updateRate>50.0</updateRate>
+          <topicName>fanuc/forcetorque</topicName>
+          <jointName>joint_6</jointName>
+      </plugin>
+  </gazebo>
 <transmission name="joint_1_tran">
     <type>transmission_interface/SimpleTransmission</type>

Commit message: fanuc simulated entire

File: fanuc_gazebo/urdf/arm_new.xacro (robot description, xacro)
@@ -224,9 +224,38 @@
     </joint>
     <!-- ROS-Industrial 'tool0' frame: all-zeros tool frame -->
-    <link name="tool0" />
-    <joint name="link_6-tool0" type="fixed">
-      <origin xyz="0 0 0" rpy="3.142 -1.571 0" />
+    <!-- <link name="tool0" /> -->
+    <joint name="grinder_joint" type="fixed">
+      <origin xyz="0 0 0" rpy="0 1.571 0" />
       <parent link="flange" />
-      <child link="tool0" />
+      <child link="tool" />
+    </joint>
+<link name="tool">
+      <inertial>
+        <mass value="4"/>
+        <origin xyz="0.0 0.0 0.0" rpy="0 0 0" />
+        <inertia
+          ixx="0.01042" ixy="0.001177" ixz="-0.0008871"
+          iyy="0.01045" iyz="0.0002226"
+          izz="0.01817"/>
+      </inertial>
+      <visual>
+        <geometry>
+          <mesh filename="package://fanuc_gazebo/mesh/grinder.stl"  scale="1.5 1.5 1.2" />
+        </geometry>
+        <material name="voilet">
+          <color rgba="1.0 0.3 1.0 1.0"/>
+        </material>
+      </visual>
+      <collision>
+        <geometry>
+          <mesh filename="package://fanuc_gazebo/mesh/grinder.stl"  scale="1.5 1.5 1.2" />
+        </geometry>
+      </collision>
+</link>
+<link name="tool_face" />
+<joint name="toolface_joint" type="fixed">
+      <origin xyz="0 0 0.33" rpy="0 -1.571 0" />
+      <parent link="tool" />
+      <child link="tool_face" />
     </joint>
 <!-- Force Torque sensor -->
@@ -327,4 +356,7 @@
       <selfCollide>true</selfCollide>
     </gazebo>
+    <gazebo reference="tool">
+      <selfCollide>true</selfCollide>
+    </gazebo>
  <!-- Gazebo colors -->
    <gazebo reference="base_link">
@@ -348,4 +380,7 @@
    <gazebo reference="link_6">
       <material>Gazebo/Orange</material>
+   </gazebo>
+   <gazebo reference="tool">
+      <material>Gazebo/Purple</material>
    </gazebo>
 <!-- Self collision in Gazebo -->

File: fanuc_gazebo/urdf/rot_base.xacro (robot description, xacro)
@@ -5,5 +5,5 @@
     <parent link="world" />
     <child link = "base_blob" />
-    <origin xyz="2.0 0 0" rpy="0.0 0.0 0" />
+    <origin xyz="2.20 0" rpy="0.0 0.0 0" />
 </joint>
     <link name="base_blob">
@@ -18,5 +18,5 @@
       <visual>
         <geometry>
-          <mesh filename="package://fanuc_gazebo/mesh/base_table.stl" scale="1 1 1"/>
+          <mesh filename="package://fanuc_gazebo/mesh/base_table.stl" scale="1 1 0.6"/>
         </geometry>
         <material name="RED">
@@ -26,5 +26,5 @@
       <collision>
         <geometry>
-          <mesh filename="package://fanuc_gazebo/mesh/base_table.stl" scale="1 1 1" />
+          <mesh filename="package://fanuc_gazebo/mesh/base_table.stl" scale="1 1 0.6" />
         </geometry>
       </collision>
@@ -48,5 +48,5 @@
       <visual>
         <geometry>
-          <mesh filename="package://fanuc_gazebo/mesh/rot_block.stl" scale="1 1 1"/>
+          <mesh filename="package://fanuc_gazebo/mesh/rot_block.stl" scale="1 1 0.6"/>
         </geometry>
         <material name="RED">
@@ -56,5 +56,5 @@
       <collision>
         <geometry>
-          <mesh filename="package://fanuc_gazebo/mesh/rot_block.stl" scale="1 1 1" />
+          <mesh filename="package://fanuc_gazebo/mesh/rot_block.stl" scale="1 1 0.6" />
         </geometry>
       </collision>

Commit message: bug fixed: interfermeter added

File: fanuc_gazebo/urdf/arm_new.xacro (robot description, xacro)
@@ -1,4 +1,5 @@
 <?xml version="1.0"?>
 <robot name="fanuc" xmlns:xacro="http://ros.org/wiki/xacro">
+<xacro:include filename="$(find fanuc_gazebo)/urdf/inter.xacro"/>
 <link name="world"/>
 <joint name="world_joint" type="fixed">
@@ -7,4 +8,65 @@
     <origin xyz="0 0 0" rpy="0.0 0.0 0" />
 </joint>
+<!-- <joint name="world_joint_base" type="fixed">
+    <parent link="world" />
+    <child link = "base_base_link" />
+    <origin xyz="3 0 0" rpy="0.0 0.0 0" />
+</joint> -->
+<!-- ###############################################################
+################################################################
+################################################################ -->
+<!-- <link name="base_base_link">
+ <inertial>
+        <mass value="0.02"/>
+        <origin xyz="0.0 0.0 0.0" rpy="0 0 0" />
+        <inertia
+          ixx="0.01042" ixy="0.001177" ixz="-0.0008871"
+          iyy="0.01045" iyz="0.0002226"
+          izz="0.01817"/>
+      </inertial>
+      <visual>
+        <geometry>
+          <cylinder length="0.05" radius="0.1"/>
+        </geometry>
+        <material name="RED">
+          <color rgba="1.0 0.0 0.0 1.0"/>
+        </material>
+      </visual>
+      <collision>
+        <geometry>
+        <cylinder length="0.00005" radius="0.00001"/>
+        </geometry>
+      </collision>
+</link> -->
+<joint name="main_inter_joint" type="prismatic">
+      <parent link="world" />
+      <child link = "interferometer" />
+      <origin xyz="3.5 0 0" rpy="0.0 0.0 1.571" />
+      <axis xyz="0 1 0" />
+      <limit lower="0" upper="1.5" effort="150.0" velocity="1.5"/>
+</joint>
+<link name="interferometer">
+      <inertial>
+        <mass value="50"/>
+        <origin xyz="0.0 0.0 0.0" rpy="0 0 0" />
+        <inertia
+          ixx="0.01042" ixy="0.001177" ixz="-0.0008871"
+          iyy="0.01045" iyz="0.0002226"
+          izz="0.01817"/>
+      </inertial>
+      <visual>
+        <geometry>
+          <mesh filename="package://fanuc_gazebo/mesh/vertical_interferometer_hbridge.stl" scale="1 1 1"/>
+        </geometry>
+        <material name="RED">
+          <color rgba="1.0 0.0 0.0 1.0"/>
+        </material>
+      </visual>
+      <collision>
+        <geometry>
+          <mesh filename="package://fanuc_gazebo/mesh/vertical_interferometer_hbridge.stl" scale="1 1 1" />
+        </geometry>
+      </collision>
+</link>
 <link name="base_link">
       <inertial>
@@ -335,28 +397,14 @@
     </actuator>
 </transmission>
-<gazebo reference="base_link">
-      <selfCollide>true</selfCollide>
-    </gazebo>
-    <gazebo reference="link_1">
-      <selfCollide>true</selfCollide>
-    </gazebo>
-    <gazebo reference="link_2">
-      <selfCollide>true</selfCollide>
-    </gazebo>
-    <gazebo reference="link_3">
-      <selfCollide>true</selfCollide>
-    </gazebo>
-    <gazebo reference="link_4">
-      <selfCollide>true</selfCollide>
-    </gazebo>
-    <gazebo reference="link_5">
-      <selfCollide>true</selfCollide>
-    </gazebo>
-    <gazebo reference="link_6">
-      <selfCollide>true</selfCollide>
-    </gazebo>
-    <gazebo reference="tool">
-      <selfCollide>true</selfCollide>
-    </gazebo>
+<transmission name="main_inter_joint_tran">
+    <type>transmission_interface/SimpleTransmission</type>
+    <joint name="main_inter_joint">
+      <hardwareInterface>hardware_interface/PositionJointInterface</hardwareInterface>
+    </joint>
+    <actuator name="main_inter_joint_motor">
+      <hardwareInterface>hardware_interface/PositionJointInterface</hardwareInterface>
+      <mechanicalReduction>1</mechanicalReduction>
+    </actuator>
+</transmission>
  <!-- Gazebo colors -->
    <gazebo reference="base_link">
@@ -382,5 +430,8 @@
    </gazebo>
    <gazebo reference="tool">
-      <material>Gazebo/Purple</material>
+      <material>Gazebo/Blue</material>
+   </gazebo>
+  <gazebo reference="interferometer">
+      <material>Gazebo/Orange</material>
    </gazebo>
 <!-- Self collision in Gazebo -->

File: fanuc_gazebo/urdf/rot_base.xacro (robot description, xacro)
@@ -60,4 +60,34 @@
       </collision>
 </link>
+<joint name="sliding_joint" type="prismatic">
+      <parent link="base_blob" />
+      <child link = "interferometer" />
+      <origin xyz="0 0 0" rpy="0.0 0.0 0.0" />
+      <axis xyz="0 0 1" />
+      <limit lower="0" upper="3.142" effort="150.0" velocity="1.5"/>
+</joint>
+<link name="interferometer">
+      <inertial>
+        <mass value="50"/>
+        <origin xyz="0.0 0.0 0.0" rpy="0 0 0" />
+        <inertia
+          ixx="0.01042" ixy="0.001177" ixz="-0.0008871"
+          iyy="0.01045" iyz="0.0002226"
+          izz="0.01817"/>
+      </inertial>
+      <visual>
+        <geometry>
+          <mesh filename="package://fanuc_gazebo/mesh/vertical_interferometer_hbridge.stl" scale="1 1 0.6"/>
+        </geometry>
+        <material name="RED">
+          <color rgba="1.0 0.0 0.0 1.0"/>
+        </material>
+      </visual>
+      <collision>
+        <geometry>
+          <mesh filename="package://fanuc_gazebo/mesh/vertical_interferometer_hbridge.stl" scale="1 1 0.6" />
+        </geometry>
+      </collision>
+</link>
 <!-- <transmission name="main_joint_tran">
     <type>transmission_interface/SimpleTransmission</type>
