Commit message: New interferometer added, everything is stable

File: fanuc_gazebo/urdf/arm_new.xacro (robot description, xacro)
@@ -1,5 +1,5 @@
 <?xml version="1.0"?>
 <robot name="fanuc" xmlns:xacro="http://ros.org/wiki/xacro">
-<xacro:include filename="$(find fanuc_gazebo)/urdf/inter.xacro"/>
+<!-- <xacro:include filename="$(find fanuc_gazebo)/urdf/inter.xacro"/> -->
 <link name="world"/>
 <joint name="world_joint" type="fixed">

File: fanuc_gazebo/urdf/inter.xacro (robot description, xacro)
@@ -1,3 +1,536 @@
 <?xml version="1.0"?>
-<robot name="fanuc"  xmlns:xacro="http://ros.org/wiki/xacro">
+<robot name="fanuc" xmlns:xacro="http://ros.org/wiki/xacro">
+<!-- <xacro:include filename="$(find fanuc_gazebo)/urdf/inter.xacro"/> -->
+<link name="world"/>
+<joint name="world_joint" type="fixed">
+    <parent link="world" />
+    <child link = "base_link" />
+    <origin xyz="0 0 0" rpy="0.0 0.0 0" />
+</joint>
+<!-- <joint name="world_joint_base" type="fixed">
+    <parent link="world" />
+    <child link = "base_base_link" />
+    <origin xyz="3 0 0" rpy="0.0 0.0 0" />
+</joint> -->
+<!-- ###############################################################
+################################################################
+################################################################ -->
+<!-- <link name="base_base_link">
+ <inertial>
+        <mass value="0.02"/>
+        <origin xyz="0.0 0.0 0.0" rpy="0 0 0" />
+        <inertia
+          ixx="0.01042" ixy="0.001177" ixz="-0.0008871"
+          iyy="0.01045" iyz="0.0002226"
+          izz="0.01817"/>
+      </inertial>
+      <visual>
+        <geometry>
+          <cylinder length="0.05" radius="0.1"/>
+        </geometry>
+        <material name="RED">
+          <color rgba="1.0 0.0 0.0 1.0"/>
+        </material>
+      </visual>
+      <collision>
+        <geometry>
+        <cylinder length="0.00005" radius="0.00001"/>
+        </geometry>
+      </collision>
+</link> -->
+<joint name="main_inter_joint" type="fixed">
+      <parent link="world" />
+      <child link = "pole" />
+      <origin xyz="2 1 0" rpy="0.0 0.0 0.0" />
+      <axis xyz="0 1 0" />
+      <limit lower="0" upper="1.5" effort="150.0" velocity="4"/>
+</joint>
+<link name="pole">
+      <inertial>
+        <mass value="50"/>
+        <origin xyz="0.0 0.0 0.0" rpy="0 0 0" />
+        <inertia
+          ixx="0.01042" ixy="0.001177" ixz="-0.0008871"
+          iyy="0.01045" iyz="0.0002226"
+          izz="0.01817"/>
+      </inertial>
+      <visual>
+        <geometry>
+          <mesh filename="package://fanuc_gazebo/mesh/pole.stl" scale="1 1 0.6"/>
+        </geometry>
+        <material name="RED">
+          <color rgba="1.0 0.0 0.0 1.0"/>
+        </material>
+      </visual>
+      <collision>
+        <geometry>
+          <mesh filename="package://fanuc_gazebo/mesh/pole.stl" scale="1 1 0.6" />
+        </geometry>
+      </collision>
+</link>
+<joint name="inter_joint_1" type="revolute">
+      <parent link="pole" />
+      <child link = "slider" />
+      <origin xyz="0 0 1.7" rpy="0.0 0.0 3.142" />
+      <axis xyz="0 0 -1" />
+      <limit lower="0" upper="3.142" effort="150.0" velocity="4"/>
+</joint>
+<link name="slider">
+      <inertial>
+        <mass value="50"/>
+        <origin xyz="0.0 0.0 0.0" rpy="0 0 0" />
+        <inertia
+          ixx="0.01042" ixy="0.001177" ixz="-0.0008871"
+          iyy="0.01045" iyz="0.0002226"
+          izz="0.01817"/>
+      </inertial>
+      <visual>
+        <geometry>
+          <mesh filename="package://fanuc_gazebo/mesh/upper_part.stl" scale="0.4 0.5 0.5"/>
+        </geometry>
+        <material name="RED">
+          <color rgba="1.0 0.0 0.0 1.0"/>
+        </material>
+      </visual>
+      <collision>
+        <geometry>
+          <mesh filename="package://fanuc_gazebo/mesh/upper_part.stl" scale="0.4 0.5 0.5" />
+        </geometry>
+      </collision>
+</link>
+<joint name="inter_joint_2" type="prismatic">
+      <parent link="slider" />
+      <child link = "module" />
+      <origin xyz="-0.4 0 0" rpy="0.0 0.0 0.0" />
+      <axis xyz="-1 0 0" />
+      <limit lower="0" upper="1.3" effort="150.0" velocity="4"/>
+</joint>
+<link name="module">
+      <inertial>
+        <mass value="50"/>
+        <origin xyz="0.0 0.0 0.0" rpy="0 0 0" />
+        <inertia
+          ixx="0.01042" ixy="0.001177" ixz="-0.0008871"
+          iyy="0.01045" iyz="0.0002226"
+          izz="0.01817"/>
+      </inertial>
+      <visual>
+        <geometry>
+          <mesh filename="package://fanuc_gazebo/mesh/vertical_interferometer_main_part.stl" scale="0.6 0.6 0.6"/>
+        </geometry>
+        <material name="RED">
+          <color rgba="1.0 0.0 0.0 1.0"/>
+        </material>
+      </visual>
+      <collision>
+        <geometry>
+          <mesh filename="package://fanuc_gazebo/mesh/vertical_interferometer_main_part.stl" scale="0.6 0.6 0.6" />
+        </geometry>
+      </collision>
+</link>
+<!-- ####################################################
+####################################################
+#################################################### -->
+<link name="base_link">
+      <inertial>
+        <mass value="1.584994"/>
+        <origin xyz="0.0 0.0 0.0" rpy="0 0 0" />
+        <inertia
+          ixx="0.01042" ixy="0.001177" ixz="-0.0008871"
+          iyy="0.01045" iyz="0.0002226"
+          izz="0.01817"/>
+      </inertial>
+      <visual>
+        <geometry>
+          <mesh filename="package://fanuc_r2000ib_support/meshes/r2000ib210f/visual/base_link.stl" scale="1 1 1"/>
+        </geometry>
+        <material name="RED">
+          <color rgba="1.0 0.0 0.0 1.0"/>
+        </material>
+      </visual>
+      <collision>
+        <geometry>
+          <mesh filename="package://fanuc_r2000ib_support/meshes/r2000ib210f/visual/base_link.stl" scale="1 1 1" />
+        </geometry>
+      </collision>
+</link>
+<joint name="joint_1" type="revolute">
+      <parent link="base_link" />
+      <child link = "link_1" />
+      <origin xyz="0 0 0.670" rpy="0.0 0.0 0.0" />
+      <axis xyz="0 0 1" />
+      <limit lower="-3.142" upper="3.142" effort="150.0" velocity="4"/>
+</joint>
+<link name="link_1">
+      <inertial>
+        <mass value="0.4"/>
+        <origin xyz="0.0 0.0 0.0" rpy="0 0 0" />
+        <inertia
+          ixx="0.01042" ixy="0.001177" ixz="-0.0008871"
+          iyy="0.01045" iyz="0.0002226"
+          izz="0.01817"/>
+      </inertial>
+      <visual>
+        <geometry>
+          <mesh filename="package://fanuc_r2000ib_support/meshes/r2000ib210f/visual/link_1.stl"  scale="1 1 1" />
+        </geometry>
+        <material name="voilet">
+          <color rgba="1.0 0.3 1.0 1.0"/>
+        </material>
+      </visual>
+      <collision>
+        <geometry>
+          <mesh filename="package://fanuc_r2000ib_support/meshes/r2000ib210f/visual/link_1.stl"  scale="1 1 1" />
+        </geometry>
+      </collision>
+</link>
+<joint name="joint_2" type="revolute">
+      <parent link="link_1" />
+      <child link = "link_2" />
+      <origin xyz="0.312 0 0" rpy="0.0 0.0 0.0" />
+      <axis xyz="0 1 0" />
+      <limit lower="-1.0472" upper="1.3264" effort="150.0" velocity="4"/>
+</joint>
+<link name="link_2">
+      <inertial>
+        <mass value="0.4"/>
+        <origin xyz="0.0 0.0 0.0" rpy="0 0 0" />
+        <inertia
+          ixx="0.01042" ixy="0.001177" ixz="-0.0008871"
+          iyy="0.01045" iyz="0.0002226"
+          izz="0.01817"/>
+      </inertial>
+      <visual>
+        <geometry>
+          <mesh filename="package://fanuc_r2000ib_support/meshes/r2000ib210f/visual/link_2.stl"  scale="1 1 1" />
+        </geometry>
+        <material name="voilet">
+          <color rgba="1.0 0.3 1.0 1.0"/>
+        </material>
+      </visual>
+      <collision>
+        <geometry>
+          <mesh filename="package://fanuc_r2000ib_support/meshes/r2000ib210f/visual/link_2.stl"  scale="1 1 1" />
+        </geometry>
+      </collision>
+</link>
+<joint name="joint_3" type="revolute">
+      <parent link="link_2" />
+      <child link = "link_3" />
+      <origin xyz="0 0 1.075" rpy="0.0 0.0 0.0" />
+      <axis xyz="0 -1 0" />
+      <limit lower="-2.303" upper="4.014" effort="150.0" velocity="4"/>
+</joint>
+<link name="link_3">
+      <inertial>
+        <mass value="0.4"/>
+        <origin xyz="0.0 0.0 0.0" rpy="0 0 0" />
+        <inertia
+          ixx="0.01042" ixy="0.001177" ixz="-0.0008871"
+          iyy="0.01045" iyz="0.0002226"
+          izz="0.01817"/>
+      </inertial>
+      <visual>
+        <geometry>
+          <mesh filename="package://fanuc_r2000ib_support/meshes/r2000ib210f/visual/link_3.stl"  scale="1 1 1" />
+        </geometry>
+        <material name="voilet">
+          <color rgba="1.0 0.3 1.0 1.0"/>
+        </material>
+      </visual>
+      <collision>
+        <geometry>
+          <mesh filename="package://fanuc_r2000ib_support/meshes/r2000ib210f/visual/link_3.stl"  scale="1 1 1" />
+        </geometry>
+      </collision>
+</link>
+<joint name="joint_4" type="revolute">
+      <parent link="link_3" />
+      <child link = "link_4" />
+      <origin xyz="0 0 0.225" rpy="0.0 0.0 0.0" />
+      <axis xyz="-1 0 0" />
+      <limit lower="-6.28" upper="6.28" effort="150.0" velocity="4"/>
+</joint>
+<link name="link_4">
+      <inertial>
+        <mass value="0.4"/>
+        <origin xyz="0.0 0.0 0.0" rpy="0 0 0" />
+        <inertia
+          ixx="0.01042" ixy="0.001177" ixz="-0.0008871"
+          iyy="0.01045" iyz="0.0002226"
+          izz="0.01817"/>
+      </inertial>
+      <visual>
+        <geometry>
+          <mesh filename="package://fanuc_r2000ib_support/meshes/r2000ib210f/visual/link_4.stl"  scale="1 1 1" />
+        </geometry>
+        <material name="voilet">
+          <color rgba="1.0 0.3 1.0 1.0"/>
+        </material>
+      </visual>
+      <collision>
+        <geometry>
+          <mesh filename="package://fanuc_r2000ib_support/meshes/r2000ib210f/visual/link_4.stl"  scale="1 1 1" />
+        </geometry>
+      </collision>
+</link>
+<joint name="joint_5" type="revolute">
+      <parent link="link_4" />
+      <child link = "link_5" />
+      <origin xyz="1.280 0 0" rpy="0.0 0.0 0.0" />
+      <axis xyz="0 -1 0" />
+      <limit lower="-2.181" upper="2.181" effort="150.0" velocity="4"/>
+</joint>
+<link name="link_5">
+      <inertial>
+<transmission name="inter_joint_1_tran">
+    <type>transmission_interface/SimpleTransmission</type>
+    <joint name="inter_joint_1">
+      <hardwareInterface>hardware_interface/PositionJointInterface</hardwareInterface>
+    </joint>
+    <actuator name="inter_joint_1_motor">
+      <hardwareInterface>hardware_interface/PositionJointInterface</hardwareInterface>
+      <mechanicalReduction>1</mechanicalReduction>
+    </actuator>
+</transmission>
+        <mass value="0.4"/>
+        <origin xyz="0.0 0.0 0.0" rpy="0 0 0" />
+        <inertia
+          ixx="0.01042" ixy="0.001177" ixz="-0.0008871"
+          iyy="0.01045" iyz="0.0002226"
+          izz="0.01817"/>
+      </inertial>
+      <visual>
+        <geometry>
+          <mesh filename="package://fanuc_r2000ib_support/meshes/r2000ib210f/visual/link_5.stl"  scale="1 1 1" />
+        </geometry>
+        <material name="voilet">
+          <color rgba="1.0 0.3 1.0 1.0"/>
+        </material>
+      </visual>
+      <collision>
+        <geometry>
+          <mesh filename="package://fanuc_r2000ib_support/meshes/r2000ib210f/visual/link_5.stl"  scale="1 1 1" />
+        </geometry>
+      </collision>
+</link>
+<joint name="joint_6" type="revolute">
+      <parent link="link_5" />
+      <child link = "link_6" />
+      <origin xyz="0.235 0 0" rpy="0.0 0.0 0.0" />
+      <axis xyz="-1 0 0" />
+      <limit lower="-6.28" upper="6.28" effort="150.0" velocity="4"/>
+</joint>
+<link name="link_6">
+      <inertial>
+        <mass value="0.4"/>
+        <origin xyz="0.0 0.0 0.0" rpy="0 0 0" />
+        <inertia
+          ixx="0.01042" ixy="0.001177" ixz="-0.0008871"
+          iyy="0.01045" iyz="0.0002226"
+          izz="0.01817"/>
+      </inertial>
+      <visual>
+        <geometry>
+          <mesh filename="package://fanuc_r2000ib_support/meshes/r2000ib210f/visual/link_6.stl"  scale="1 1 1" />
+        </geometry>
+        <material name="voilet">
+          <color rgba="1.0 0.3 1.0 1.0"/>
+        </material>
+      </visual>
+      <collision>
+        <geometry>
+          <mesh filename="package://fanuc_r2000ib_support/meshes/r2000ib210f/visual/link_6.stl"  scale="1 1 1" />
+        </geometry>
+      </collision>
+</link>
+    <link name="base" />
+    <joint name="base_link-base" type="fixed">
+      <origin xyz="0 0 0.670" rpy="0 0 0"/>
+      <parent link="base_link"/>
+      <child link="base"/>
+    </joint>
+    <!-- ROS-Industrial 'flange' frame: attachment point for EEF models -->
+    <link name="flange" />
+    <joint name="joint_6-flange" type="fixed">
+      <origin xyz="0 0 0" rpy="0 0 0" />
+      <parent link="link_6" />
+      <child link="flange" />
+    </joint>
+    <!-- ROS-Industrial 'tool0' frame: all-zeros tool frame -->
+    <!-- <link name="tool0" /> -->
+    <joint name="grinder_joint" type="fixed">
+      <origin xyz="0 0 0" rpy="0 1.571 0" />
+      <parent link="flange" />
+      <child link="tool" />
+    </joint>
+<link name="tool">
+      <inertial>
+        <mass value="4"/>
+        <origin xyz="0.0 0.0 0.0" rpy="0 0 0" />
+        <inertia
+          ixx="0.01042" ixy="0.001177" ixz="-0.0008871"
+          iyy="0.01045" iyz="0.0002226"
+          izz="0.01817"/>
+      </inertial>
+      <visual>
+        <geometry>
+          <mesh filename="package://fanuc_gazebo/mesh/grinder.stl"  scale="1.5 1.5 1.2" />
+        </geometry>
+        <material name="voilet">
+          <color rgba="1.0 0.3 1.0 1.0"/>
+        </material>
+      </visual>
+      <collision>
+        <geometry>
+          <mesh filename="package://fanuc_gazebo/mesh/grinder.stl"  scale="1.5 1.5 1.2" />
+        </geometry>
+      </collision>
+</link>
+<link name="tool_face" />
+<joint name="toolface_joint" type="fixed">
+      <origin xyz="0 0 0.33" rpy="0 -1.571 0" />
+      <parent link="tool" />
+      <child link="tool_face" />
+    </joint>
+<!-- Force Torque sensor -->
+<gazebo reference="joint_6">
+      <provideFeedback>true</provideFeedback>
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